Commit message: trav grid: Mid-360 Risley sim + real-robot calibration + CNN traversability fusion
Three improvements wired together for the 3D-frontier exploration pipeline.

1) Mid-360 sim densification (Livox Risley CSV replay)
   Replaced the uniform-grid raycast in mujoco_ros2_control's lidar_sensor
   with replay of Livox-SDK's official Mid-360 non-repetitive scan pattern
   (mid360.csv, 800k samples = 4s of azimuth/zenith). Defaults: 20k rays
   per frame + σ=2cm Gaussian range noise. Resolution + density now match
   the real Mid-360; nvblox walls fill all z-layers correctly.
   Env overrides: MUJOCO_LIDAR_SCAN_PATTERN_CSV (empty=uniform-grid fall
   back), MUJOCO_LIDAR_RAYS_PER_FRAME, MUJOCO_LIDAR_NOISE_STDDEV_M.

2) Mid-360 mount calibration on every sim TF source
   Updated all MJCFs (18), both go2w xacros, the go2w.urdf snapshot,
   pointlio_gazebo*.yaml extrinsics, the gbplanner3 sim static TF
   publisher, and the gbplanner3 demo3 launcher to the real-robot
   calibration measured 2026-04-17: roll=-0.036809 rad (-2.11°),
   pitch=+0.263591 rad (+15.10°), yaw=0. MJCFs use quat=(0.99116,
   -0.01824, 0.13139, 0.00242) to match ROS Rz·Ry·Rx convention. The
   prior 13° pitch-only guess gave sim a 2° tilted elevation map that
   never appeared on the real robot.

3) ETH CNN traversability re-enabled on Blackwell + ramp-safe fusion
   The Phase-3.3 patch had disabled the elevation_mapping_cupy CNN
   because torch.cat lacks an sm_120 cubin. Added get_filter_cupy() —
   a 65-line pure-cupy reimplementation of the 3-branch dilated 3x3
   conv stack — and a runtime backend selector that picks it on
   compute_capability >= 10 (Blackwell). Float32 match vs numpy
   reference < 1e-7. CNN now populates the `traversability` layer at
   ~5 Hz and correctly marks wall TOPS as lethal (not just the 1-cell
   rim that the analytical step_residual filter caught).

   The CNN over-rejects ramps (training set was mostly flat ground),
   so the grid_map_filters chain now also computes:
     slope_margin  = clamp((0.5236 - slope) / 0.5236, 0, 1)
     step_margin   = clamp((0.06 - step_residual) / 0.06, 0, 1)
     ramp_safe     = clamp(slope_margin * step_margin * 100, 0, 1)
     trav_fused    = max(traversability, ramp_safe)
   On a 14° ramp: ramp_safe=0.998, fused mean=0.999. On walls (slope
   >57°): ramp_safe=0, fused=raw CNN (still lethal). On flat ground:
   both 1.0. Live numbers from demo_ramp:
     ramp:  CNN lethal 91 -> fused lethal 9 (out of 1012 eligible)
     wall:  CNN lethal 1834 -> fused lethal 1834 (preserved)
     flat:  CNN lethal 452 -> fused lethal 0 (noise cleaned)
   Nav2 reads trav_fused; raw CNN and analytical trav_eth remain as
   parallel comparison layers visible in RViz.

Also fixed grid_map_filters.yaml filter contiguity: filter9b..9e and
filter23a/b had to be renumbered because filters::FilterChain silently
drops non-integer-suffix keys (see memory note).

RViz nav_test.rviz: added 4 GridMap displays (trav_fused, raw CNN,
trav_eth, slope_cost, step_cost) under the existing root, defaulting
to trav_fused so the visualization matches what Nav2 consumes.

Co-Authored-By: Claude Opus 4.7 (1M context) <noreply@anthropic.com>

File: src/go2w/go2_gazebo_sim/mujoco/go2w.urdf (robot description, URDF)
Before this commit: robot go2w_description, 37 links, 36 joints
Joints:
- joint livox_mid360_base_joint: origin xyz=0.1870 0 0.0803 rpy=0 0.2269 0 -> xyz=0.1870 0 0.0803 rpy=-0.036809 0.263591 0

File: src/go2w/go2_gazebo_sim/urdf/go2w/livox_mid360.xacro (robot description, xacro)
@@ -4,7 +4,8 @@
   <!--
     Livox MID-360 LiDAR Macro for go2w_description
-    Based on official Unitree Go2 MID-360 mounting specifications:
+    Mounting on the Go2W (real-robot calibrated 2026-04-17, see
+    scripts/real/onboard_fastlio_noetic.sh:262):
     - Position in IMU frame: (0.1870, 0, 0.0803) meters
-    - Rotation: 13° around Y-axis (0.2269 radians)
+    - Rotation: pitch +0.263591 rad (+15.10°), roll -0.036809 rad (-2.11°), yaw 0
     NOTE: This macro uses the accurate MID-360 mesh (mid-360.dae).
     Usage:
@@ -44,10 +45,12 @@
       <child link="${name}_base"/>
       <!--
-        Official Unitree Go2 MID-360 transform from IMU frame:
-        - Translation: (0.1870, 0, 0.0803) meters
-        - Rotation: 13° around Y-axis (pitch)
-        - This matches the transformation matrix from documentation
+        Real-robot calibrated Mid-360 mount on the Go2W (measured 2026-04-17).
+        Translation: (0.1870, 0, 0.0803) m from the IMU frame.
+        Rotation: roll=-0.036809 rad (-2.11°), pitch=+0.263591 rad (+15.10°), yaw=0.
+        Mirrors scripts/real/onboard_fastlio_noetic.sh:262. The prior 13°
+        pitch-only value was a documentation guess that drifted ~2° from
+        real measurement; sim and real now share the same TF tilt.
       -->
-      <origin xyz="0.1870 0 0.0803" rpy="0 0.2269 0"/>
+      <origin xyz="0.1870 0 0.0803" rpy="-0.036809 0.263591 0"/>
     </joint>
     <!-- LiDAR Optical Frame (sensor frame for point cloud) -->

File: src/go2w/unitree_go2w_ros2/src/go2w_description/urdf/livox_mid360.xacro (robot description, xacro)
@@ -3,7 +3,8 @@
   <!--
     Livox MID-360 LiDAR Macro for go2w_description
-    Based on official Unitree Go2 MID-360 mounting specifications:
+    Mounting on the Go2W (real-robot calibrated 2026-04-17, see
+    scripts/real/onboard_fastlio_noetic.sh:262):
     - Position in IMU frame: (0.1870, 0, 0.0803) meters
-    - Rotation: 13° around Y-axis (0.2269 radians)
+    - Rotation: pitch +0.263591 rad (+15.10°), roll -0.036809 rad (-2.11°), yaw 0
     NOTE: This macro uses the accurate MID-360 mesh (mid-360.dae).
     Usage:
@@ -43,10 +44,14 @@
       <child link="${name}_base"/>
       <!--
-        Official Unitree Go2 MID-360 transform from IMU frame:
-        - Translation: (0.1870, 0, 0.0803) meters
-        - Rotation: 13° around Y-axis (pitch)
-        - This matches the transformation matrix from documentation
+        Real-robot calibrated Mid-360 mount on the Go2W (measured 2026-04-17).
+        Translation: (0.1870, 0, 0.0803) m from the IMU frame.
+        Rotation: roll=-0.036809 rad (-2.11°), pitch=+0.263591 rad (+15.10°), yaw=0.
+        Sourced from scripts/real/onboard_fastlio_noetic.sh:262 (the static
+        map→camera_init TF that Fast-LIO consumes on real hardware). The
+        prior value (rpy="0 0.2269 0", 13° pitch only) was a documentation
+        guess that drifted ~2° from real and gave sim a tilted elevation
+        map that didn't appear on the real robot.
       -->
-      <origin xyz="0.1870 0 0.0803" rpy="0 0.2269 0"/>
+      <origin xyz="0.1870 0 0.0803" rpy="-0.036809 0.263591 0"/>
     </joint>
     <!-- LiDAR Optical Frame (sensor frame for point cloud) -->
